File: Tastatur.kicad_pcb (KiCad board)
At the start: 2 copper layers, 175.3 x 134 mm, 140 parts, among them J1 USB_C_Receptacle_USB2.0_16P, U2 Pico

Commit message: change dm dp
Connections:
- J1 pad A6: DM -> DP
- J1 pad A7: DP -> DM
- J1 pad B6: DM -> DP
- J1 pad B7: DP -> DM
- TP1 pad 1: DP -> DM
- TP2 pad 1: DM -> DP
Routing:
- net DP: track 18.6 -> 15.7 mm
- net DM: track 15.7 -> 18.6 mm
