File: Tastatur.kicad_sch (KiCad schematic)
At the start: 139 parts, among them J1 USB_C_Receptacle_USB2.0_16P, U2 Pico

Commit message: change dm dp
Connections:
- net DM: now also J1.A7 (D-), J1.B7 (D-), TP1.1; no longer J1.A6 (D+), J1.B6 (D+), TP2.1
- net DP: now also J1.A6 (D+), J1.B6 (D+), TP2.1; no longer J1.A7 (D-), J1.B7 (D-), TP1.1
Changed lines of the file:
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@@
 	(global_label "DM"
 		(shape input)
-		(at 63.5 73.66 0)
+		(at 63.5 63.5 0)
 		(fields_autoplaced yes)
 		(effects
@@
 		)
 		(property "Intersheetrefs" "${INTERSHEET_REFS}"
-			(at 69.2066 73.66 0)
+			(at 69.2066 63.5 0)
 			(effects
 				(font
@@
 	(global_label "DP"
 		(shape input)
-		(at 63.5 63.5 0)
+		(at 63.5 73.66 0)
 		(fields_autoplaced yes)
 		(effects
@@
 		)
 		(property "Intersheetrefs" "${INTERSHEET_REFS}"
-			(at 69.0252 63.5 0)
+			(at 69.0252 73.66 0)
 			(effects
 				(font
